Commit message: deleted link2

File: rrbot_description/urdf/myrobot.xacro (robot description, xacro)
@@ -6,6 +6,6 @@
   <xacro:property name="mass" value="1" /> <!-- arbitrary value for mass -->
   <xacro:property name="width" value="0.1" /> <!-- Square dimensions (widthxwidth) of beams -->
-  <xacro:property name="height1" value="2" /> <!-- Link 1 -->
-  <xacro:property name="height2" value="5" /> <!-- Link 2 -->
+  <xacro:property name="height1" value="0.6" /> <!-- Link 1 -->
+  <!--<xacro:property name="height2" value="5" /> Link 2 -->
   <xacro:property name="height3" value="1" /> <!-- Link 3 -->
   <xacro:property name="camera_link" value="0.05" /> <!-- Size of square 'camera' box -->
@@ -47,11 +47,11 @@
   <joint name="joint1" type="fixed">
     <parent link="link1"/>
-    <child link="link2"/>
-    <origin xyz="0 ${width} ${height1 - axel_offset}" rpy="0 1.5 0"/>
+    <child link="link3"/>
+    <origin xyz="0 ${width} ${height1 - axel_offset}" rpy="0 1.5708 0"/>
     <axis xyz="0 1 0"/>
     <dynamics damping="0.7"/>
   </joint>
   <!-- Middle Link -->
-  <link name="link2">
+ <!--  <link name="link2">
     <collision>
       <origin xyz="0 0 ${height2/2 - axel_offset}" rpy="0 0 0"/>
@@ -59,6 +59,6 @@
 	<box size="${width} ${width} ${height2}"/>
       </geometry>
-    </collision>
-    <visual>
+    </collision> -->
+    <!-- <visual>
       <origin xyz="0 0 ${height2/2 - axel_offset}" rpy="0 0 0"/>
       <geometry>
@@ -75,6 +75,6 @@
 	  izz="${mass / 12.0 * (width*width + width*width)}"/>
     </inertial>
-  </link>
-  <joint name="joint2" type="fixed">
+  </link> -->
+ <!--  <joint name="joint2" type="fixed">
     <parent link="link2"/>
     <child link="link3"/>
@@ -82,5 +82,5 @@
     <axis xyz="0 1 0"/>
     <dynamics damping="0.7"/>
-  </joint>
+  </joint> -->
   <!-- Top Link -->
   <link name="link3">

Commit message: changed the postition of the laserscan

File: rrbot_description/urdf/myrobot.xacro (robot description, xacro)
@@ -109,5 +109,5 @@
   <joint name="hokuyo_joint" type="fixed">
     <axis xyz="0 1 0" />
-    <origin xyz="0 0 ${height3 - axel_offset/2}" rpy="0 0 0"/>
+    <origin xyz="0 ${-axel_offset-0.02} ${height3 - axel_offset*2}" rpy="1.5708 0 0"/>
     <parent link="link3"/>
     <child link="hokuyo_link"/>

Commit message: decrease height1

File: rrbot_description/urdf/myrobot.xacro (robot description, xacro)
@@ -6,5 +6,5 @@
   <xacro:property name="mass" value="1" /> <!-- arbitrary value for mass -->
   <xacro:property name="width" value="0.1" /> <!-- Square dimensions (widthxwidth) of beams -->
-  <xacro:property name="height1" value="0.6" /> <!-- Link 1 -->
+  <xacro:property name="height1" value="0.5" /> <!-- Link 1 -->
   <!--<xacro:property name="height2" value="5" /> Link 2 -->
   <xacro:property name="height3" value="1" /> <!-- Link 3 -->

Commit message: change geometry to match real model

File: rrbot_description/urdf/myrobot.xacro (robot description, xacro)
@@ -6,7 +6,7 @@
   <xacro:property name="mass" value="1" /> <!-- arbitrary value for mass -->
   <xacro:property name="width" value="0.1" /> <!-- Square dimensions (widthxwidth) of beams -->
-  <xacro:property name="height1" value="0.5" /> <!-- Link 1 -->
+  <xacro:property name="height1" value="0.55" /> <!-- Link 1 -->
   <!--<xacro:property name="height2" value="5" /> Link 2 -->
-  <xacro:property name="height3" value="1" /> <!-- Link 3 -->
+  <xacro:property name="height3" value="0.7" /> <!-- Link 3 -->
   <xacro:property name="camera_link" value="0.05" /> <!-- Size of square 'camera' box -->
   <xacro:property name="axel_offset" value="0.05" /> <!-- Space btw top of beam and the each joint -->

Commit message: adjusted camera block

File: rrbot_description/urdf/myrobot.xacro (robot description, xacro)
@@ -148,9 +148,9 @@
     </collision>
     <visual>
-      <origin xyz="0 0 0" rpy="0 0 0"/>
+      <origin xyz="0 0 0" rpy="0 ${PI/2} 0"/>
       <geometry>
-	<box size="${camera_link} ${camera_link} ${camera_link}"/>
+	<cylinder radius="${camera_link/3}" length="${camera_link/2}"/>
       </geometry>
-      <material name="red"/>
+      <material name="black"/>
     </visual>
     <inertial>
